Commit message: adding bouding box for the "robot". looks way more stable now. need to tune mass, spring and damping + fix wheel sprink back position

File: urdf/robot.urdf (robot description, URDF)
Before this commit: robot robot, 14 links, 13 joints
Links:
- link base_link: geometry collision box size=2.5 0.75 0.1; visual box size=2.5 0.75 0.1
- link fourcheBL: geometry collision box size=0.5 0.1 0.1; visual box size=0.5 0.1 0.1
- link fourcheBR: geometry collision box size=0.5 0.1 0.1; visual box size=0.5 0.1 0.1
- link fourcheFL: geometry collision box size=0.5 0.1 0.1; visual box size=0.5 0.1 0.1
- link fourcheFR: geometry collision box size=0.5 0.1 0.1; visual box size=0.5 0.1 0.1
- link hipBL: geometry collision box size=1 0.1 0.1; visual box size=1 0.1 0.1
- link hipBR: geometry collision box size=1 0.1 0.1; visual box size=1 0.1 0.1
- link hipFL: geometry collision box size=1 0.1 0.1; visual box size=1 0.1 0.1
- link hipFR: geometry collision box size=1 0.1 0.1; visual box size=1 0.1 0.1
- link wheelBL: geometry collision cylinder length=0.05 radius=0.4; visual cylinder length=0.05 radius=0.4
- link wheelBR: geometry collision cylinder length=0.05 radius=0.4; visual cylinder length=0.05 radius=0.4
- link wheelFL: geometry collision cylinder length=0.05 radius=0.4; visual cylinder length=0.05 radius=0.4
- link wheelFR: geometry collision cylinder length=0.05 radius=0.4; visual cylinder length=0.05 radius=0.4

Commit message: round URDF value

File: urdf/robot.urdf (robot description, URDF)
Before this commit: robot robot, 14 links, 13 joints
Links:
- link base_link: mass 1 -> 100
Joints:
- joint base_link_to_hipBL: axis -0.01199487623111348 -0.9998443265953507 0.012940074160918302 -> 0 -1 0
- joint base_link_to_hipBR: axis -0.01199487623111348 -0.9998443265953507 0.012940074160918302 -> 0 -1 0
- joint base_link_to_hipFL: axis -0.011994876231113505 -0.9998443265953507 0.012940074160918299 -> 0 -1 0
- joint base_link_to_hipFR: axis -0.01199487623111348 -0.9998443265953507 0.012940074160918302 -> 0 -1 0
- joint fourcheBL_to_wheelBL: axis 0 0.9999984826271444 0.0017420514943473635 -> 0 1 0
- joint fourcheBR_to_wheelBR: axis 0 0.9999984826271444 0.0017420514943473635 -> 0 1 0
- joint fourcheFL_to_wheelFL: axis 0 0.9999984826271444 0.001742051494347363 -> 0 1 0
- joint fourcheFR_to_wheelFR: axis 0 0.9999984826271444 0.0017420514943473635 -> 0 1 0
- joint hipBL_to_fourcheBL: axis -0.999980271823115 -0.0029739561465167465 0.005532770500197626 -> -1 0 0
- joint hipBR_to_fourcheBR: axis -0.999980271823115 -0.0029739561465167465 0.005532770500197626 -> -1 0 0
- joint hipFL_to_fourcheFL: axis -0.9999802718231151 -0.0029739561465120046 0.005532770500188856 -> -1 0 0
- joint hipFR_to_fourcheFR: axis -0.999980271823115 -0.0029739561465167465 0.005532770500197626 -> -1 0 0

Commit message: robot is stable on the floor. damping was too low

File: urdf/robot.urdf (robot description, URDF)
Before this commit: robot robot, 14 links, 13 joints
Links:
- link fourcheBL: mass 1 -> 5
- link fourcheBR: mass 1 -> 5
- link fourcheFL: mass 1 -> 5
- link fourcheFR: mass 1 -> 5
- link hipBL: mass 1 -> 5
- link hipBR: mass 1 -> 5
- link hipFL: mass 1 -> 5
- link hipFR: mass 1 -> 5
- link wheelBL: mass 1 -> 5
- link wheelBR: mass 1 -> 5
- link wheelFL: mass 1 -> 5
- link wheelFR: mass 1 -> 5

Commit message: the vehicule roll "straight" but require some parameters tunning

File: urdf/robot.urdf (robot description, URDF)
Before this commit: robot robot, 14 links, 13 joints
Joints:
- joint fourcheBL_to_wheelBL: origin xyz=-0.25 0.075 0 rpy=0 0 0 -> xyz=-0.25 0 0 rpy=0 0 0
- joint fourcheBR_to_wheelBR: origin xyz=-0.25 -0.07 0 rpy=0 0 0 -> xyz=-0.25 0 0 rpy=0 0 0
- joint fourcheFL_to_wheelFL: origin xyz=0.25 0.075 0 rpy=0 0 0 -> xyz=0.25 0 0 rpy=0 0 0
- joint fourcheFR_to_wheelFR: origin xyz=0.25 -0.07 0 rpy=0 0 0 -> xyz=0.25 0 0 rpy=0 0 0

Commit message: defined heightfield differently. collision check is now correct

File: urdf/robot.urdf (robot description, URDF)
Before this commit: robot robot, 14 links, 13 joints
Joints:
- joint base_joint: origin xyz=0.009466139050656165 0 1 rpy=0 0 0 -> xyz=0 0 1 rpy=0 0 0

Commit message: implemented 3 wheel variant to simplify. still unable to turn :(

File: urdf/robot.urdf (robot description, URDF)
Before this commit: robot robot, 14 links, 13 joints
Links:
- link wheelBL: mass 5 -> 10
- link wheelBR: mass 5 -> 10
- link wheelFL: mass 5 -> 10
