Commit message: added more geometry since there seems to be a flaw with the pivot design

File: urdf/robotPivotThreeWheel.urdf (robot description, URDF)
Before this commit: robot robot, 10 links, 9 joints
Joints:
- joint fourcheFL_to_wheelFL: origin xyz=0.25 0 0 rpy=1.570796326794897 0 0 -> xyz=0.25 0 -0.1 rpy=1.570796326794897 0 0
- joint fourcheFR_to_wheelFR: origin xyz=0.25 0 0 rpy=1.570796326794897 0 0 -> xyz=0.25 0 -0.1 rpy=1.570796326794897 0 0
