Commit message: I really wish I had the time to make a controller :(

File: urdf/robotLinearThreeWheel.urdf (robot description, URDF)
Before this commit: robot robot, 14 links, 13 joints
Links:
- link feetB: geometry visual box size=0.1 0.1 0.4
- link feetFL: geometry visual box size=0.1 0.1 0.4
- link feetFR: geometry visual box size=0.1 0.1 0.4
Joints:
- joint feetB_to_wheelB: limit lower=-1 upper=1 effort=1000.0 velocity=0.5 -> 
- joint feetFL_to_wheelFL: limit lower=-1 upper=1 effort=1000.0 velocity=0.5 -> 
- joint feetFR_to_wheelFR: limit lower=-1 upper=1 effort=1000.0 velocity=0.5 -> 
- joint hipFL_to_legFL: limit lower=-1 upper=1 effort=1000.0 velocity=0.5 -> lower=-1 upper=1
- joint hipFR_to_legFR: limit lower=-1 upper=1 effort=1000.0 velocity=0.5 -> lower=-1 upper=1
