Commit message: added tool to compute tip angle

File: urdf/robotLinearFourWheel.urdf (robot description, URDF)
Before this commit: robot robot, 18 links, 17 joints
Links:
- link feetBL: geometry visual box size=0.1 0.1 0.4
- link feetBR: geometry visual box size=0.1 0.1 0.4
- link feetFL: geometry visual box size=0.1 0.1 0.4
- link feetFR: geometry visual box size=0.1 0.1 0.4
Joints:
- joint feetBL_to_wheelBL: limit lower=-1 upper=1 effort=1000.0 velocity=0.5 -> 
- joint feetBR_to_wheelBR: limit lower=-1 upper=1 effort=1000.0 velocity=0.5 -> 
- joint feetFL_to_wheelFL: limit lower=-1 upper=1 effort=1000.0 velocity=0.5 -> 
- joint feetFR_to_wheelFR: limit lower=-1 upper=1 effort=1000.0 velocity=0.5 -> 
- joint hipBL_to_legBL: limit lower=-1 upper=1 effort=1000.0 velocity=0.5 -> lower=-1 upper=1
- joint hipBR_to_legBR: limit lower=-1 upper=1 effort=1000.0 velocity=0.5 -> lower=-1 upper=1
- joint hipFL_to_legFL: limit lower=-1 upper=1 effort=1000.0 velocity=0.5 -> lower=-1 upper=1
- joint hipFR_to_legFR: limit lower=-1 upper=1 effort=1000.0 velocity=0.5 -> lower=-1 upper=1
- joint legBL_to_feetBL: limit lower=-1 upper=1 effort=1000.0 velocity=0.5 -> lower=-1 upper=1
- joint legBR_to_feetBR: limit lower=-1 upper=1 effort=1000.0 velocity=0.5 -> lower=-1 upper=1
- joint legFL_to_feetFL: limit lower=-1 upper=1 effort=1000.0 velocity=0.5 -> lower=-1 upper=1
- joint legFR_to_feetFR: limit lower=-1 upper=1 effort=1000.0 velocity=0.5 -> lower=-1 upper=1
